File: PowerProtection.sch (KiCad schematic (older format))
At the start: 7 parts, among them K1 G6SK-2

Commit message: Il reste a trouver empreintes et router
Parts:
- removed D2: D, LIB_BE_PHELMA_CMS:LED_1206_3216Metric_Pad1.42x1.75mm_HandSolder, symbol Device:D
- added D8: 10V, symbol Device:D_Zener
- added Q1: IPB110P06LM, Package_TO_SOT_SMD:TO-263-3_TabPin2, symbol Transistor_FET:IRF7606PBF
- added R7: 10k, symbol Device:R
Connections:
- wire segments 45 -> 36
Other:
- note added: "Reverse polarity protection"
Changed lines of the file:
@@
 $Descr A4 11693 8268
 encoding utf-8
-Sheet 2 3
+Sheet 2 2
 Title ""
 Date ""
@@
 Wire Wire Line
 	9100 3450 9100 3550
-Wire Wire Line
-	9450 3450 9450 3550
 Connection ~ 9100 3050
-Wire Wire Line
-	9450 3050 9450 3150
-Wire Wire Line
-	9100 3050 9450 3050
 Connection ~ 8750 3050
 Wire Wire Line
@@
 AR Path="/5F8230FD" Ref="#PWR?"  Part="1"
 AR Path="/5F802FB9/5F8230FD" Ref="#PWR03"  Part="1"
-F 0 "#PWR03" H 8750 3300 50  0001 C CNN
+F 0 "#PWR?" H 8750 3300 50  0001 C CNN
 F 1 "GND" H 8755 3377 50  0000 C CNN
 F 2 "" H 8750 3550 50  0001 C CNN
@@
 AR Path="/5F823103" Ref="#PWR?"  Part="1"
 AR Path="/5F802FB9/5F823103" Ref="#PWR04"  Part="1"
-F 0 "#PWR04" H 9100 3700 50  0001 C CNN
+F 0 "#PWR?" H 9100 3700 50  0001 C CNN
 F 1 "GND" H 9105 3777 50  0000 C CNN
 F 2 "" H 9100 3950 50  0001 C CNN
@@
 	1    9100 3950
 	1    0    0    -1
-$EndComp
-$Comp
-L power:GND #PWR?
-U 1 1 5F823109
-P 9450 3550
-AR Path="/5F823109" Ref="#PWR?"  Part="1"
-AR Path="/5F802FB9/5F823109" Ref="#PWR027"  Part="1"
-F 0 "#PWR027" H 9450 3300 50  0001 C CNN
-F 1 "GND" H 9455 3377 50  0000 C CNN
-F 2 "" H 9450 3550 50  0001 C CNN
-F 3 "" H 9450 3550 50  0001 C CNN
-	1    9450 3550
-	1    0    0    -1
-$EndComp
-$Comp
-L Device:D D?
-U 1 1 5F82310F
-P 9450 3300
-AR Path="/5F82310F" Ref="D?"  Part="1"
-AR Path="/5F802FB9/5F82310F" Ref="D2"  Part="1"
-F 0 "D2" V 9404 3379 50  0000 L CNN
-F 1 "D" V 9495 3379 50  0000 L CNN
-F 2 "LIB_BE_PHELMA_CMS:LED_1206_3216Metric_Pad1.42x1.75mm_HandSolder" H 9450 3300 50  0001 C CNN
-F 3 "~" H 9450 3300 50  0001 C CNN
-	1    9450 3300
-	0    1    1    0
 $EndComp
 $Comp
@@
 AR Path="/5F823115" Ref="D?"  Part="1"
 AR Path="/5F802FB9/5F823115" Ref="D1"  Part="1"
-F 0 "D1" V 9139 3583 50  0000 R CNN
+F 0 "D?" V 9139 3583 50  0000 R CNN
 F 1 "LED" V 9048 3583 50  0000 R CNN
 F 2 "LIB_BE_PHELMA_CMS:LED_1206_3216Metric_Pad1.42x1.75mm_HandSolder" H 9100 3700 50  0001 C CNN
@@
 AR Path="/5F82311B" Ref="R?"  Part="1"
 AR Path="/5F802FB9/5F82311B" Ref="R1"  Part="1"
-F 0 "R1" H 9170 3346 50  0000 L CNN
+F 0 "R?" H 9170 3346 50  0000 L CNN
 F 1 "R" H 9170 3255 50  0000 L CNN
 F 2 "LIB_BE_PHELMA_CMS:R_1206_3216Metric_Pad1.42x1.75mm_HandSolder" V 9030 3300 50  0001 C CNN
@@
 AR Path="/5F823121" Ref="C?"  Part="1"
 AR Path="/5F802FB9/5F823121" Ref="C2"  Part="1"
-F 0 "C2" H 8868 3346 50  0000 L CNN
+F 0 "C?" H 8868 3346 50  0000 L CNN
 F 1 "CP" H 8868 3255 50  0000 L CNN
 F 2 "LIB_BE_PHELMA_CMS:C_1206_3216Metric_Pad1.42x1.75mm_HandSolder" H 8788 3150 50  0001 C CNN
@@
 AR Path="/5F823127" Ref="F?"  Part="1"
 AR Path="/5F802FB9/5F823127" Ref="F1"  Part="1"
-F 0 "F1" H 8460 3096 50  0000 L CNN
+F 0 "F?" H 8460 3096 50  0000 L CNN
 F 1 "Fuse" H 8460 3005 50  0000 L CNN
 F 2 "" V 8330 3050 50  0001 C CNN
@@
 	0    -1   -1   0
 $EndComp
-Connection ~ 9450 3050
 Text HLabel 10050 3050 2    50   Output ~ 0
 ProtectedPowerOut+
-Wire Wire Line
-	9450 3050 10050 3050
 $Comp
 L Relay:G6SK-2 K1
 U 1 1 5F83DBFF
 P 3300 4300
-F 0 "K1" V 2433 4300 50  0000 C CNN
+F 0 "K?" V 2433 4300 50  0000 C CNN
 F 1 "G6SK-2" V 2524 4300 50  0000 C CNN
 F 2 "" H 3850 4250 50  0001 L CNN
@@
 U 1 1 5F8833FD
 P 2750 3600
-F 0 "C1" H 2865 3646 50  0000 L CNN
+F 0 "C?" H 2865 3646 50  0000 L CNN
 F 1 "C" H 2865 3555 50  0000 L CNN
 F 2 "LIB_BE_PHELMA_CMS:C_1206_3216Metric_Pad1.42x1.75mm_HandSolder" H 2788 3450 50  0001 C CNN
@@
 Wire Wire Line
 	3600 4300 4100 4300
-Wire Wire Line
-	4100 4300 4100 4100
 $Comp
 L power:GND #PWR?
 U 1 1 5FAC711C
-P 2900 4600
+P 2500 4600
 AR Path="/5FAC711C" Ref="#PWR?"  Part="1"
 AR Path="/5F802FB9/5FAC711C" Ref="#PWR0101"  Part="1"
-F 0 "#PWR0101" H 2900 4350 50  0001 C CNN
-F 1 "GND" H 2905 4427 50  0000 C CNN
-F 2 "" H 2900 4600 50  0001 C CNN
-F 3 "" H 2900 4600 50  0001 C CNN
-	1    2900 4600
+F 0 "#PWR?" H 2500 4350 50  0001 C CNN
+F 1 "GND" H 2505 4427 50  0000 C CNN
+F 2 "" H 2500 4600 50  0001 C CNN
+F 3 "" H 2500 4600 50  0001 C CNN
+	1    2500 4600
 	0    1    1    0
 $EndComp
@@
 L power:GND #PWR?
 U 1 1 5FAC7686
-P 3700 4700
+P 4100 4700
 AR Path="/5FAC7686" Ref="#PWR?"  Part="1"
 AR Path="/5F802FB9/5FAC7686" Ref="#PWR0102"  Part="1"
-F 0 "#PWR0102" H 3700 4450 50  0001 C CNN
-F 1 "GND" H 3705 4527 50  0000 C CNN
-F 2 "" H 3700 4700 50  0001 C CNN
-F 3 "" H 3700 4700 50  0001 C CNN
-	1    3700 4700
+F 0 "#PWR?" H 4100 4450 50  0001 C CNN
+F 1 "GND" H 4105 4527 50  0000 C CNN
+F 2 "" H 4100 4700 50  0001 C CNN
+F 3 "" H 4100 4700 50  0001 C CNN
+	1    4100 4700
 	0    -1   -1   0
 $EndComp
@@
 L power:GND #PWR?
 U 1 1 5FAC7C37
-P 3700 4500
+P 4100 4500
 AR Path="/5FAC7C37" Ref="#PWR?"  Part="1"
 AR Path="/5F802FB9/5FAC7C37" Ref="#PWR0103"  Part="1"
-F 0 "#PWR0103" H 3700 4250 50  0001 C CNN
-F 1 "GND" H 3705 4327 50  0000 C CNN
-F 2 "" H 3700 4500 50  0001 C CNN
-F 3 "" H 3700 4500 50  0001 C CNN
-	1    3700 4500
-	0    -1   -1   0
-$EndComp
-Wire Wire Line
-	3000 4600 2900 4600
-Wire Wire Line
-	3600 4500 3700 4500
-Wire Wire Line
-	3700 4700 3600 4700
-Text HLabel 4150 3950 2    50   Input ~ 0
+F 0 "#PWR?" H 4100 4250 50  0001 C CNN
+F 1 "GND" H 4105 4327 50  0000 C CNN
+F 2 "" H 4100 4500 50  0001 C CNN
+F 3 "" H 4100 4500 50  0001 C CNN
+	1    4100 4500
+	0    -1   -1   0
+$EndComp
+Text HLabel 4150 4100 2    50   Input ~ 0
 BatteryPowerIn-
 Wire Wire Line
-	3600 3950 3600 4100
-Wire Wire Line
-	3600 3950 4150 3950
-$Sheet
-S 4900 2850 2200 900
-U 5FBB308A
-F0 "XavProtec" 50
-F1 "XavProtec.sch" 50
-F2 "PowerIn+" I L 4900 3000 50
-F3 "PowerIn-" I L 4900 3550 50
-F4 "PowerOut+" O R 7100 3000 50
-F5 "PowerOut-" O R 7100 3550 50
-$EndSheet
-Wire Wire Line
-	8250 3050 7350 3050
-Wire Wire Line
-	7350 3050 7350 2950
-Wire Wire Line
-	7350 2950 7100 2950
-Wire Wire Line
-	7100 2950 7100 3000
-Wire Wire Line
-	7100 3550 7700 3550
-Wire Wire Line
-	7700 3550 7700 4400
-Wire Wire Line
-	7700 4400 10100 4400
-Wire Wire Line
-	10100 4400 10100 4100
-Wire Wire Line
-	2250 3050 4800 3050
-Wire Wire Line
-	4800 3050 4800 3000
-Wire Wire Line
-	4800 3000 4900 3000
-Wire Wire Line
-	4900 3550 4300 3550
-Wire Wire Line
-	4300 3550 4300 4100
-Wire Wire Line
-	4300 4100 4100 4100
+	3600 4100 4150 4100
+$Comp
+L power:GND #PWR?
+U 1 1 5F8A11CB
+P 4100 4300
+AR Path="/5F8A11CB" Ref="#PWR?"  Part="1"
+AR Path="/5F802FB9/5F8A11CB" Ref="#PWR0105"  Part="1"
+F 0 "#PWR?" H 4100 4050 50  0001 C CNN
+F 1 "GND" H 4105 4127 50  0000 C CNN
+F 2 "" H 4100 4300 50  0001 C CNN
+F 3 "" H 4100 4300 50  0001 C CNN
+	1    4100 4300
+	0    -1   -1   0
+$EndComp
+$Comp
+L power:GND #PWR?
+U 1 1 5F8A37D8
+P 10050 4100
+AR Path="/5F8A37D8" Ref="#PWR?"  Part="1"
+AR Path="/5F802FB9/5F8A37D8" Ref="#PWR0106"  Part="1"
+F 0 "#PWR?" H 10050 3850 50  0001 C CNN
+F 1 "GND" H 10055 3927 50  0000 C CNN
+F 2 "" H 10050 4100 50  0001 C CNN
+F 3 "" H 10050 4100 50  0001 C CNN
+	1    10050 4100
+	0    1    1    0
+$EndComp
+Wire Wire Line
+	10100 4100 10050 4100
+Wire Wire Line
+	2500 4600 3000 4600
+Wire Wire Line
+	3600 4700 4100 4700
+Wire Wire Line
+	3600 4500 4100 4500
+$Comp
+L Transistor_FET:IRF7606PBF Q?
+U 1 1 5F88E169
+P 5900 3150
+AR Path="/5F88E169" Ref="Q?"  Part="1"
+AR Path="/5F898EC7/5F88E169" Ref="Q?"  Part="1"
+AR Path="/5F802FB9/5FBB308A/5F88E169" Ref="Q?"  Part="1"
+AR Path="/5F802FB9/5F88E169" Ref="Q1"  Part="1"
+F 0 "Q?" V 6242 3150 50  0000 C CNN
+F 1 "IPB110P06LM" V 6151 3150 50  0000 C CNN
+F 2 "Package_TO_SOT_SMD:TO-263-3_TabPin2" H 6100 3075 50  0001 L CIN
+F 3 "https://www.infineon.com/dgdl/Infineon-IPB110P06LM-DS-v02_00-EN.pdf?fileId=5546d46269e1c019016a03e2d06000ae" V 5900 3150 50  0001 L CNN
+	1    5900 3150
+	0    -1   -1   0
+$EndComp
+$Comp
+L Device:D_Zener D?
+U 1 1 5F88E16F
+P 6250 3250
+AR Path="/5F88E16F" Ref="D?"  Part="1"
+AR Path="/5F898EC7/5F88E16F" Ref="D?"  Part="1"
+AR Path="/5F802FB9/5FBB308A/5F88E16F" Ref="D?"  Part="1"
+AR Path="/5F802FB9/5F88E16F" Ref="D8"  Part="1"
+F 0 "D?" V 6204 3330 50  0000 L CNN
+F 1 "10V" V 6295 3330 50  0000 L CNN
+F 2 "" H 6250 3250 50  0001 C CNN
+F 3 "~" H 6250 3250 50  0001 C CNN
+	1    6250 3250
+	0    1    1    0
+$EndComp
+$Comp
+L Device:R R?
+U 1 1 5F88E175
+P 5900 3700
+AR Path="/5F88E175" Ref="R?"  Part="1"
+AR Path="/5F898EC7/5F88E175" Ref="R?"  Part="1"
+AR Path="/5F802FB9/5FBB308A/5F88E175" Ref="R?"  Part="1"
+AR Path="/5F802FB9/5F88E175" Ref="R7"  Part="1"
+F 0 "R?" H 5970 3746 50  0000 L CNN
+F 1 "10k" H 5970 3655 50  0000 L CNN
+F 2 "" V 5830 3700 50  0001 C CNN
+F 3 "~" H 5900 3700 50  0001 C CNN
+	1    5900 3700
+	1    0    0    -1
+$EndComp
+Wire Wire Line
+	6250 3450 5900 3450
+Wire Wire Line
+	5900 3450 5900 3350
+Wire Wire Line
+	5900 3450 5900 3550
+Connection ~ 5900 3450
+$Comp
+L power:GND #PWR?
+U 1 1 5F88E180
+P 5900 3950
+AR Path="/5F88E180" Ref="#PWR?"  Part="1"
+AR Path="/5F898EC7/5F88E180" Ref="#PWR?"  Part="1"
+AR Path="/5F802FB9/5FBB308A/5F88E180" Ref="#PWR?"  Part="1"
+AR Path="/5F802FB9/5F88E180" Ref="#PWR028"  Part="1"
+F 0 "#PWR?" H 5900 3700 50  0001 C CNN
+F 1 "GND" H 5905 3777 50  0000 C CNN
+F 2 "" H 5900 3950 50  0001 C CNN
+F 3 "" H 5900 3950 50  0001 C CNN
+	1    5900 3950
+	1    0    0    -1
+$EndComp
+Wire Wire Line
+	5900 3850 5900 3950
+Wire Wire Line
+	6250 3400 6250 3450
+Wire Wire Line
+	6100 3050 6250 3050
+Wire Wire Line
+	6250 3100 6250 3050
+Connection ~ 6250 3050
+Wire Wire Line
+	2250 3050 5700 3050
+Wire Wire Line
+	6250 3050 8250 3050
+Wire Notes Line
+	5350 2650 5350 4300
+Wire Notes Line
+	5350 4300 6500 4300
+Wire Notes Line
+	6500 4300 6500 2650
+Wire Notes Line
+	6500 2650 5350 2650
+Text Notes 5350 4400 0    50   ~ 0
+Reverse polarity protection
+Wire Wire Line
+	9100 3050 10050 3050
 $EndSCHEMATC

Commit message: ajout de la tirette
Changed lines of the file:
@@
 AR Path="/5F8230FD" Ref="#PWR?"  Part="1"
 AR Path="/5F802FB9/5F8230FD" Ref="#PWR03"  Part="1"
-F 0 "#PWR?" H 8750 3300 50  0001 C CNN
+F 0 "#PWR03" H 8750 3300 50  0001 C CNN
 F 1 "GND" H 8755 3377 50  0000 C CNN
 F 2 "" H 8750 3550 50  0001 C CNN
@@
 AR Path="/5F823103" Ref="#PWR?"  Part="1"
 AR Path="/5F802FB9/5F823103" Ref="#PWR04"  Part="1"
-F 0 "#PWR?" H 9100 3700 50  0001 C CNN
+F 0 "#PWR04" H 9100 3700 50  0001 C CNN
 F 1 "GND" H 9105 3777 50  0000 C CNN
 F 2 "" H 9100 3950 50  0001 C CNN
@@
 AR Path="/5F823115" Ref="D?"  Part="1"
 AR Path="/5F802FB9/5F823115" Ref="D1"  Part="1"
-F 0 "D?" V 9139 3583 50  0000 R CNN
+F 0 "D1" V 9139 3583 50  0000 R CNN
 F 1 "LED" V 9048 3583 50  0000 R CNN
 F 2 "LIB_BE_PHELMA_CMS:LED_1206_3216Metric_Pad1.42x1.75mm_HandSolder" H 9100 3700 50  0001 C CNN
@@
 AR Path="/5F82311B" Ref="R?"  Part="1"
 AR Path="/5F802FB9/5F82311B" Ref="R1"  Part="1"
-F 0 "R?" H 9170 3346 50  0000 L CNN
+F 0 "R1" H 9170 3346 50  0000 L CNN
 F 1 "R" H 9170 3255 50  0000 L CNN
 F 2 "LIB_BE_PHELMA_CMS:R_1206_3216Metric_Pad1.42x1.75mm_HandSolder" V 9030 3300 50  0001 C CNN
@@
 AR Path="/5F823121" Ref="C?"  Part="1"
 AR Path="/5F802FB9/5F823121" Ref="C2"  Part="1"
-F 0 "C?" H 8868 3346 50  0000 L CNN
+F 0 "C2" H 8868 3346 50  0000 L CNN
 F 1 "CP" H 8868 3255 50  0000 L CNN
 F 2 "LIB_BE_PHELMA_CMS:C_1206_3216Metric_Pad1.42x1.75mm_HandSolder" H 8788 3150 50  0001 C CNN
@@
 AR Path="/5F823127" Ref="F?"  Part="1"
 AR Path="/5F802FB9/5F823127" Ref="F1"  Part="1"
-F 0 "F?" H 8460 3096 50  0000 L CNN
+F 0 "F1" H 8460 3096 50  0000 L CNN
 F 1 "Fuse" H 8460 3005 50  0000 L CNN
 F 2 "" V 8330 3050 50  0001 C CNN
@@
 U 1 1 5F83DBFF
 P 3300 4300
-F 0 "K?" V 2433 4300 50  0000 C CNN
+F 0 "K1" V 2433 4300 50  0000 C CNN
 F 1 "G6SK-2" V 2524 4300 50  0000 C CNN
 F 2 "" H 3850 4250 50  0001 L CNN
@@
 U 1 1 5F8833FD
 P 2750 3600
-F 0 "C?" H 2865 3646 50  0000 L CNN
+F 0 "C1" H 2865 3646 50  0000 L CNN
 F 1 "C" H 2865 3555 50  0000 L CNN
 F 2 "LIB_BE_PHELMA_CMS:C_1206_3216Metric_Pad1.42x1.75mm_HandSolder" H 2788 3450 50  0001 C CNN
@@
 AR Path="/5FAC711C" Ref="#PWR?"  Part="1"
 AR Path="/5F802FB9/5FAC711C" Ref="#PWR0101"  Part="1"
-F 0 "#PWR?" H 2500 4350 50  0001 C CNN
+F 0 "#PWR0101" H 2500 4350 50  0001 C CNN
 F 1 "GND" H 2505 4427 50  0000 C CNN
 F 2 "" H 2500 4600 50  0001 C CNN
@@
 AR Path="/5FAC7686" Ref="#PWR?"  Part="1"
 AR Path="/5F802FB9/5FAC7686" Ref="#PWR0102"  Part="1"
-F 0 "#PWR?" H 4100 4450 50  0001 C CNN
+F 0 "#PWR0102" H 4100 4450 50  0001 C CNN
 F 1 "GND" H 4105 4527 50  0000 C CNN
 F 2 "" H 4100 4700 50  0001 C CNN
@@
 AR Path="/5FAC7C37" Ref="#PWR?"  Part="1"
 AR Path="/5F802FB9/5FAC7C37" Ref="#PWR0103"  Part="1"
-F 0 "#PWR?" H 4100 4250 50  0001 C CNN
+F 0 "#PWR0103" H 4100 4250 50  0001 C CNN
 F 1 "GND" H 4105 4327 50  0000 C CNN
 F 2 "" H 4100 4500 50  0001 C CNN
@@
 AR Path="/5F8A11CB" Ref="#PWR?"  Part="1"
 AR Path="/5F802FB9/5F8A11CB" Ref="#PWR0105"  Part="1"
-F 0 "#PWR?" H 4100 4050 50  0001 C CNN
+F 0 "#PWR0105" H 4100 4050 50  0001 C CNN
 F 1 "GND" H 4105 4127 50  0000 C CNN
 F 2 "" H 4100 4300 50  0001 C CNN
@@
 AR Path="/5F8A37D8" Ref="#PWR?"  Part="1"
 AR Path="/5F802FB9/5F8A37D8" Ref="#PWR0106"  Part="1"
-F 0 "#PWR?" H 10050 3850 50  0001 C CNN
+F 0 "#PWR0106" H 10050 3850 50  0001 C CNN
 F 1 "GND" H 10055 3927 50  0000 C CNN
 F 2 "" H 10050 4100 50  0001 C CNN
@@
 AR Path="/5F802FB9/5FBB308A/5F88E169" Ref="Q?"  Part="1"
 AR Path="/5F802FB9/5F88E169" Ref="Q1"  Part="1"
-F 0 "Q?" V 6242 3150 50  0000 C CNN
+F 0 "Q1" V 6242 3150 50  0000 C CNN
 F 1 "IPB110P06LM" V 6151 3150 50  0000 C CNN
 F 2 "Package_TO_SOT_SMD:TO-263-3_TabPin2" H 6100 3075 50  0001 L CIN
@@
 AR Path="/5F802FB9/5FBB308A/5F88E16F" Ref="D?"  Part="1"
 AR Path="/5F802FB9/5F88E16F" Ref="D8"  Part="1"
-F 0 "D?" V 6204 3330 50  0000 L CNN
+F 0 "D8" V 6204 3330 50  0000 L CNN
 F 1 "10V" V 6295 3330 50  0000 L CNN
 F 2 "" H 6250 3250 50  0001 C CNN
@@
 AR Path="/5F802FB9/5FBB308A/5F88E175" Ref="R?"  Part="1"
 AR Path="/5F802FB9/5F88E175" Ref="R7"  Part="1"
-F 0 "R?" H 5970 3746 50  0000 L CNN
+F 0 "R7" H 5970 3746 50  0000 L CNN
 F 1 "10k" H 5970 3655 50  0000 L CNN
 F 2 "" V 5830 3700 50  0001 C CNN
@@
 AR Path="/5F802FB9/5FBB308A/5F88E180" Ref="#PWR?"  Part="1"
 AR Path="/5F802FB9/5F88E180" Ref="#PWR028"  Part="1"
-F 0 "#PWR?" H 5900 3700 50  0001 C CNN
+F 0 "#PWR028" H 5900 3700 50  0001 C CNN
 F 1 "GND" H 5905 3777 50  0000 C CNN
 F 2 "" H 5900 3950 50  0001 C CNN
